Commit message: [urdf] Add wall behind the robot.

File: urdf/demo.urdf.xacro (robot description, xacro)
@@ -6,3 +6,4 @@
                       joint_limits="${xacro.load_yaml('$(find franka_description)/robots/panda/joint_limits.yaml')}">
   </xacro:franka_robot>
+  <!-- wall behind the table -->
 </robot>

File: urdf/support.urdf.xacro (robot description, xacro)
@@ -33,4 +33,23 @@
         </collision>
       </link>
+      <link name="wall_link">
+        <inertial>
+          <mass value="200"/>
+          <origin xyz="0 0 1."/>
+          <inertia ixx="50"  ixy="0"  ixz="0" iyy="50" iyz="0" izz="50" />
+        </inertial>
+        <visual>
+          <origin xyz="0 0 1.0"/>
+          <geometry>
+            <box size="3.0 0.1 2.0"/>
+          </geometry>
+        </visual>
+        <collision>
+          <origin xyz="0 0 1.0"/>
+          <geometry>
+            <box size="3.0 0.1 2.0"/>
+          </geometry>
+        </collision>
+      </link>
       <!-- Gazebo requires a joint to a link called "world" for statically mounted robots -->
       <link name="world" />
@@ -45,4 +64,9 @@
         <child  link="$(arg arm_id)_link0" />
       </joint>
+      <joint name="wall_joint" type="fixed">
+        <origin xyz="0 1.07 0" />
+        <parent link="world"/>
+        <child link="wall_link"/>
+      </joint>
   </xacro:macro>
 </robot>

Commit message: Change name to support dual arm manipulation

File: urdf/demo.urdf.xacro (robot description, xacro)
@@ -1,9 +1,8 @@
 <?xml version='1.0' encoding='utf-8'?>
-<robot xmlns:xacro="http://www.ros.org/wiki/xacro" name="panda">
+<robot xmlns:xacro="http://www.ros.org/wiki/xacro" name="pandas">
   <xacro:include filename="$(find agimus_demos)/franka/manipulation/urdf/franka_robot.xacro"/>
   <xacro:include filename="$(find agimus_demos)/franka/manipulation/urdf/support.urdf.xacro"/>
   <xacro:support/>
-  <xacro:arg name="arm_id" default="panda" />
-  <xacro:franka_robot arm_id="$(arg arm_id)"
+  <xacro:franka_robot arm_id="panda1"
                       joint_limits="${xacro.load_yaml('$(find franka_description)/robots/panda/joint_limits.yaml')}">
   </xacro:franka_robot>

File: urdf/franka_hand.xacro (robot description, xacro)
@@ -2,5 +2,5 @@
 <robot xmlns:xacro="http://www.ros.org/wiki/xacro" name="hand">
   <!-- safety_distance: Minimum safety distance in [m] by which the collision volumes are expanded and which is enforced during robot motions -->
-  <xacro:macro name="franka_hand" params="connected_to:='' arm_id:='panda' rpy:='0 0 0' xyz:='0 0 0' tcp_xyz:='0 0 0.1034' tcp_rpy:='0 0 0' safety_distance:=0 gazebo:=false description_pkg:=franka_description">
+  <xacro:macro name="franka_hand" params="connected_to:='' arm_id rpy:='0 0 0' xyz:='0 0 0' tcp_xyz:='0 0 0.1034' tcp_rpy:='0 0 0' safety_distance:=0 gazebo:=false description_pkg:=franka_description">
     <xacro:unless value="${connected_to == ''}">
       <joint name="${arm_id}_hand_joint" type="fixed">

File: urdf/franka_robot.xacro (robot description, xacro)
@@ -3,6 +3,4 @@
   <xacro:macro name="franka_robot" params="arm_id joint_limits">
     <!-- Name of this panda -->
-    <!-- Should a franka_gripper be mounted at the flange?" -->
-    <xacro:arg name="hand" default="true" />
     <!-- Positional offset between $(arm_id)_hand -> $(arm_id)_hand_tcp [m]. Only used when hand:=true -->
     <xacro:arg name="tcp_xyz" default="0 0 0.1034" />
@@ -13,17 +11,15 @@
     <xacro:include filename="$(find franka_description)/robots/common/utils.xacro" />
     <xacro:include filename="$(find franka_description)/robots/common/franka_arm.xacro" />
+    <xacro:include filename="$(find agimus_demos)/franka/manipulation/urdf/franka_hand.xacro"/>
     <xacro:franka_arm arm_id="${arm_id}" safety_distance="0.03" gazebo="$(arg gazebo)" joint_limits="${joint_limits}"/>
-    <xacro:if value="$(arg hand)">
-      <xacro:include filename="$(find agimus_demos)/franka/manipulation/urdf/franka_hand.xacro"/>
-      <xacro:franka_hand
-          arm_id="$(arg arm_id)"
-          rpy="0 0 ${-pi/4}"
-          tcp_xyz="$(arg tcp_xyz)"
-          tcp_rpy="$(arg tcp_rpy)"
-          connected_to="$(arg arm_id)_link8"
-          safety_distance="0.03"
-          gazebo="$(arg gazebo)"
-       />
-    </xacro:if>
+    <xacro:franka_hand
+        arm_id="${arm_id}"
+        rpy="0 0 ${-pi/4}"
+        tcp_xyz="$(arg tcp_xyz)"
+        tcp_rpy="$(arg tcp_rpy)"
+        connected_to="${arm_id}_link8"
+        safety_distance="0.03"
+        gazebo="$(arg gazebo)"
+        />
     <!-- Define additional Gazebo tags -->
     <xacro:if value="$(arg gazebo)">
@@ -56,11 +52,9 @@
          tip="${arm_id}_joint8"
        />
-      <xacro:if value="$(arg hand)">
-        <xacro:gazebo-joint joint="${arm_id}_finger_joint1" transmission="hardware_interface/EffortJointInterface" />
-        <xacro:gazebo-joint joint="${arm_id}_finger_joint2" transmission="hardware_interface/EffortJointInterface" />
-        <!-- Friction specific material for Rubber/Rubber contact -->
-        <xacro:gazebo-friction link="${arm_id}_leftfinger" mu="1.13" />
-        <xacro:gazebo-friction link="${arm_id}_rightfinger" mu="1.13" />
-      </xacro:if>
+      <xacro:gazebo-joint joint="${arm_id}_finger_joint1" transmission="hardware_interface/EffortJointInterface" />
+      <xacro:gazebo-joint joint="${arm_id}_finger_joint2" transmission="hardware_interface/EffortJointInterface" />
+      <!-- Friction specific material for Rubber/Rubber contact -->
+      <xacro:gazebo-friction link="${arm_id}_leftfinger" mu="1.13" />
+      <xacro:gazebo-friction link="${arm_id}_rightfinger" mu="1.13" />
       <gazebo>
         <plugin name="gazebo_ros_control" filename="libgazebo_ros_control.so">

File: urdf/support.urdf.xacro (robot description, xacro)
@@ -62,5 +62,5 @@
         <origin xyz="-0.5365 0.2215 .78" rpy="0 0 0" />
         <parent link="support_link" />
-        <child  link="$(arg arm_id)_link0" />
+        <child  link="panda1_link0" />
       </joint>
       <joint name="wall_joint" type="fixed">

Commit message: Add calibration chessboard when argument calibration is set to true

File: urdf/demo.urdf.xacro (robot description, xacro)
@@ -1,7 +1,8 @@
 <?xml version='1.0' encoding='utf-8'?>
 <robot xmlns:xacro="http://www.ros.org/wiki/xacro" name="pandas">
+  <arg name="calibration" default="false"/>
   <xacro:include filename="$(find agimus_demos)/franka/manipulation/urdf/franka_robot.xacro"/>
   <xacro:include filename="$(find agimus_demos)/franka/manipulation/urdf/support.urdf.xacro"/>
-  <xacro:support/>
+  <xacro:support chessboard="$(arg calibration)"/>
   <xacro:franka_robot arm_id="panda1"
                       joint_limits="${xacro.load_yaml('$(find franka_description)/robots/panda/joint_limits.yaml')}">

File: urdf/support.urdf.xacro (robot description, xacro)
@@ -1,5 +1,5 @@
 <?xml version='1.0' encoding='utf-8'?>
 <robot xmlns:xacro="http://www.ros.org/wiki/xacro">
-  <xacro:macro name="support">
+  <xacro:macro name="support" params="chessboard">
       <link name="support_link">
         <inertial>
@@ -32,4 +32,13 @@
           </geometry>
         </collision>
+        <xacro:if value="${chessboard}">
+          <!-- calibration chessboard-->
+          <visual>
+            <origin xyz="0 0 .761" rpy="0 0 0"/>
+            <geometry>
+	      <mesh filename="package://gerard_bauzil/meshes/visp/chessboard-10-7.dae" scale="0.027 0.027 1."/>
+            </geometry>
+          </visual>
+        </xacro:if>
       </link>
       <link name="wall_link">

Commit message: Use panda2 robot.

File: urdf/demo.urdf.xacro (robot description, xacro)
@@ -4,5 +4,5 @@
   <xacro:include filename="$(find agimus_demos)/franka/manipulation/urdf/support.urdf.xacro"/>
   <xacro:support/>
-  <xacro:franka_robot arm_id="panda1"
+  <xacro:franka_robot arm_id="panda2"
                       joint_limits="${xacro.load_yaml('$(find franka_description)/robots/panda/joint_limits.yaml')}">
   </xacro:franka_robot>

File: urdf/support.urdf.xacro (robot description, xacro)
@@ -20,5 +20,5 @@
           </geometry>
         </collision>
-        <visual>
+        <!--visual>
           <origin xyz="-0.61 0.2215 0.77"/>
           <geometry>
@@ -30,4 +30,16 @@
           <geometry>
 	    <box size="0.363 0.252 0.02"/>
+          </geometry>
+        </collision-->
+        <visual>
+          <origin xyz="0.6385 -0.1655 0.77"/>
+          <geometry>
+            <box size="0.3 0.3 0.02"/>
+          </geometry>
+        </visual>
+        <collision>
+          <origin xyz="0.6385 -0.1655 0.77"/>
+          <geometry>
+            <box size="0.3 0.3 0.02"/>
           </geometry>
         </collision>
@@ -52,4 +64,27 @@
         </collision>
       </link>
+      <!-- Wrap panda1 robot into a box shaped obstacle -->
+      <link name="panda1_box">
+        <inertial>
+          <mass value="100"/>
+          <origin xyz="0 0 0"/>
+          <inertia ixx="25"  ixy="0"  ixz="0" iyy="25" iyz="0" izz="25" />
+        </inertial>
+        <collision>
+          <origin xyz="0 0 0"/>
+          <geometry>
+            <box size="0.44 0.803 0.80"/>
+          </geometry>
+        </collision>
+        <visual>
+          <origin xyz="0 0 0"/>
+          <geometry>
+            <box size="0.44 0.803 0.80"/>
+          </geometry>
+          <material name="lightGrey">
+            <color rgba="0.9 0.9 0.9 0.5"/>
+          </material>
+        </visual>
+      </link>
       <!-- Gazebo requires a joint to a link called "world" for statically mounted robots -->
       <link name="world" />
@@ -60,7 +95,7 @@
       </joint>
       <joint name="support_joint" type="fixed">
-        <origin xyz="-0.5365 0.2215 .78" rpy="0 0 0" />
+        <origin xyz="0.563 -0.1655 .78" rpy="0 0 ${pi}" />
         <parent link="support_link" />
-        <child  link="panda1_link0" />
+        <child  link="panda2_link0" />
       </joint>
       <joint name="wall_joint" type="fixed">
@@ -69,4 +104,9 @@
         <child link="wall_link"/>
       </joint>
+      <joint name="panda1_box_joint" type="fixed">
+        <origin xyz="-0.6315 0 1.17" />
+        <parent link="world"/>
+        <child link="panda1_box"/>
+      </joint>
   </xacro:macro>
 </robot>

Commit message: Remove calibration option in launch and xacro files
  Calibration chessboard will be added as an object.

File: urdf/demo.urdf.xacro (robot description, xacro)
@@ -1,8 +1,7 @@
 <?xml version='1.0' encoding='utf-8'?>
 <robot xmlns:xacro="http://www.ros.org/wiki/xacro" name="pandas">
-  <arg name="calibration" default="false"/>
   <xacro:include filename="$(find agimus_demos)/franka/manipulation/urdf/franka_robot.xacro"/>
   <xacro:include filename="$(find agimus_demos)/franka/manipulation/urdf/support.urdf.xacro"/>
-  <xacro:support chessboard="$(arg calibration)"/>
+  <xacro:support/>
   <xacro:franka_robot arm_id="panda1"
                       joint_limits="${xacro.load_yaml('$(find franka_description)/robots/panda/joint_limits.yaml')}">

File: urdf/support.urdf.xacro (robot description, xacro)
@@ -1,5 +1,5 @@
 <?xml version='1.0' encoding='utf-8'?>
 <robot xmlns:xacro="http://www.ros.org/wiki/xacro">
-  <xacro:macro name="support" params="chessboard">
+  <xacro:macro name="support" params="">
       <link name="support_link">
         <inertial>
@@ -32,13 +32,4 @@
           </geometry>
         </collision>
-        <xacro:if value="${chessboard}">
-          <!-- calibration chessboard-->
-          <visual>
-            <origin xyz="0 0 .761" rpy="0 0 0"/>
-            <geometry>
-	      <mesh filename="package://gerard_bauzil/meshes/visp/chessboard-10-7.dae" scale="0.027 0.027 1."/>
-            </geometry>
-          </visual>
-        </xacro:if>
       </link>
       <link name="wall_link">
