Commit message: [urdf] Add second wall and obstacle in the corner.

File: urdf/support.urdf.xacro (robot description, xacro)
@@ -45,5 +45,5 @@
         </collision>
       </link>
-      <link name="wall_link">
+      <link name="wall_link_1">
         <inertial>
           <mass value="200"/>
@@ -61,4 +61,45 @@
           <geometry>
             <box size="3.0 0.1 2.0"/>
+          </geometry>
+        </collision>
+      </link>
+      <link name="wall_link_2">
+        <inertial>
+          <mass value="200"/>
+          <origin xyz="0 0 1."/>
+          <inertia ixx="50"  ixy="0"  ixz="0" iyy="50" iyz="0" izz="50" />
+        </inertial>
+        <visual>
+          <origin xyz="0 0 1.0"/>
+          <geometry>
+            <box size="0.1 2.0 2.0"/>
+          </geometry>
+          <material name="lightGrey">
+            <color rgba="0.9 0.9 0.9 0.5"/>
+          </material>
+        </visual>
+        <collision>
+          <origin xyz="0 0 1.0"/>
+          <geometry>
+            <box size="0.1 2.0 2.0"/>
+          </geometry>
+        </collision>
+      </link>
+      <link name="wall_link_3">
+        <inertial>
+          <mass value="200"/>
+          <origin xyz="0 0 1."/>
+          <inertia ixx="50"  ixy="0"  ixz="0" iyy="50" iyz="0" izz="50" />
+        </inertial>
+        <visual>
+          <origin xyz="0 0 1.0"/>
+          <geometry>
+            <box size="0.7 0.12 2.0"/>
+          </geometry>
+        </visual>
+        <collision>
+          <origin xyz="0 0 1.0"/>
+          <geometry>
+            <box size="0.7 0.12 2.0"/>
           </geometry>
         </collision>
@@ -99,8 +140,18 @@
         <child  link="panda2_link0" />
       </joint>
-      <joint name="wall_joint" type="fixed">
+      <joint name="wall_joint_1" type="fixed">
         <origin xyz="0 1.07 0" />
         <parent link="world"/>
-        <child link="wall_link"/>
+        <child link="wall_link_1"/>
+      </joint>
+      <joint name="wall_joint_2" type="fixed">
+        <origin xyz="1.78 0 0" />
+        <parent link="world"/>
+        <child link="wall_link_2"/>
+      </joint>
+      <joint name="wall_joint_3" type="fixed">
+        <origin xyz="1.40 0.96 0" />
+        <parent link="world"/>
+        <child link="wall_link_3"/>
       </joint>
       <joint name="panda1_box_joint" type="fixed">

Commit message: [urdf] Add a pedestal to put the part on.

File: urdf/support.urdf.xacro (robot description, xacro)
@@ -105,4 +105,23 @@
         </collision>
       </link>
+      <link name="pedestal">
+        <inertial>
+          <mass value="1."/>
+          <origin xyz="1.05 0.45 0.4625"/>
+          <inertia ixx=".01" iyy=".01" izz=".1" ixy="0" ixz="0" iyz="0"/>
+        </inertial>
+        <visual>
+          <origin xyz="0 0 0.4625"/>
+          <geometry>
+            <box size="0.25 0.25 0.925"/>
+          </geometry>
+        </visual>
+        <collision>
+          <origin xyz="0 0 0.4625"/>
+          <geometry>
+            <box size="0.25 0.25 0.925"/>
+          </geometry>
+        </collision>
+      </link>
       <!-- Wrap panda1 robot into a box shaped obstacle -->
       <link name="panda1_box">
@@ -155,4 +174,9 @@
         <child link="wall_link_3"/>
       </joint>
+      <joint name="pedestal_joint" type="fixed">
+        <origin xyz="1.05 0.45 0"/>
+        <parent link="world"/>
+        <child link="pedestal"/>
+      </joint>
       <joint name="panda1_box_joint" type="fixed">
         <origin xyz="-0.6315 0 1.17" />
