Commit message: [urdf] Remove self-collision geometries.

File: urdf/utils.xacro (robot description, xacro)
@@ -50,16 +50,4 @@
       </xacro:if>
     </link>
-    <!-- sub-link defining coarse geometries of real robot's internal self-collision -->
-    <link name="${prefix}${name}_sc">
-      <xacro:unless value="${gazebo}">
-        <xacro:insert_block name="self_collision_geometries" />
-      </xacro:unless>
-    </link>
-    <!-- fixed joint between both sub-links -->
-    <joint name="${prefix}${name}_sc_joint" type="fixed">
-      <origin rpy="${rpy}" />
-      <parent link="${prefix}${name}" />
-      <child link="${prefix}${name}_sc" />
-    </joint>
   </xacro:macro>
   <!-- =========================================================== -->

Commit message: [srdf] Reintroduce self collision geometries
  Deactivate collisions with part with a SRDF string
  It seems that on the robot, collisions are detected online using the self
  collision geometries. Using standard geometries for self collision produces
  trajectories that are detected in collision by the robot.

File: urdf/utils.xacro (robot description, xacro)
@@ -50,4 +50,16 @@
       </xacro:if>
     </link>
+    <!-- sub-link defining coarse geometries of real robot's internal self-collision -->
+    <link name="${prefix}${name}_sc">
+      <xacro:unless value="${gazebo}">
+        <xacro:insert_block name="self_collision_geometries" />
+      </xacro:unless>
+    </link>
+    <!-- fixed joint between both sub-links -->
+    <joint name="${prefix}${name}_sc_joint" type="fixed">
+      <origin rpy="${rpy}" />
+      <parent link="${prefix}${name}" />
+      <child link="${prefix}${name}_sc" />
+    </joint>
   </xacro:macro>
   <!-- =========================================================== -->
