Commit message: Start implementing manipulation planning problem
  - fix collision model: handle self-collision geometries that have been
    added in the urdf file,
  - add a small box.
  - start script_hpp.py.

File: urdf/franka_robot.xacro (robot description, xacro)
@@ -4,5 +4,5 @@
     <!-- Name of this panda -->
     <!-- Should a franka_gripper be mounted at the flange?" -->
-    <xacro:arg name="hand" default="false" />
+    <xacro:arg name="hand" default="true" />
     <!-- Positional offset between $(arm_id)_hand -> $(arm_id)_hand_tcp [m]. Only used when hand:=true -->
     <xacro:arg name="tcp_xyz" default="0 0 0.1034" />
@@ -15,5 +15,5 @@
     <xacro:franka_arm arm_id="${arm_id}" safety_distance="0.03" gazebo="$(arg gazebo)" joint_limits="${joint_limits}"/>
     <xacro:if value="$(arg hand)">
-      <xacro:include filename="$(find franka_description)/robots/common/franka_hand.xacro"/>
+      <xacro:include filename="$(find agimus_demos)/franka/manipulation/urdf/franka_hand.xacro"/>
       <xacro:franka_hand
           arm_id="$(arg arm_id)"
@@ -26,47 +26,6 @@
        />
     </xacro:if>
-      <link name="support_link">
-        <inertial>
-          <mass value="200"/>
-          <origin xyz="0 0 0.45"/>
-          <inertia ixx="50"  ixy="0"  ixz="0" iyy="50" iyz="0" izz="50" />
-        </inertial>
-        <visual>
-          <origin xyz="0 0 0.38"/>
-          <geometry>
-	    <box size="1.703 0.803 0.76"/>
-          </geometry>
-        </visual>
-        <collision>
-          <origin xyz="0 0 0.38"/>
-          <geometry>
-	    <box size="1.703 0.803 0.76"/>
-          </geometry>
-        </collision>
-        <visual>
-          <origin xyz="-0.61 0.2215 0.77"/>
-          <geometry>
-	    <box size="0.363 0.252 0.02"/>
-          </geometry>
-        </visual>
-        <collision>
-          <origin xyz="-0.61 0.2215 0.77"/>
-          <geometry>
-	    <box size="0.363 0.252 0.02"/>
-          </geometry>
-        </collision>
-      </link>
-      <!-- Gazebo requires a joint to a link called "world" for statically mounted robots -->
-      <link name="world" />
-      <joint name="world_joint" type="fixed">
-        <origin xyz="0 0 0" rpy="0 0 0" />
-        <parent link="world" />
-        <child  link="support_link" />
-      </joint>
-      <joint name="support_joint" type="fixed">
-        <origin xyz="-0.5365 0.2215 .78" rpy="0 0 0" />
-        <parent link="support_link" />
-        <child  link="$(arg arm_id)_link0" />
-      </joint>
+    <xacro:include filename="$(find agimus_demos)/franka/manipulation/urdf/support.urdf.xacro"/>
+    <xacro:support/>
     <!-- Define additional Gazebo tags -->
     <xacro:if value="$(arg gazebo)">

Commit message: Add camera D435.

File: urdf/franka_robot.xacro (robot description, xacro)
@@ -22,4 +22,33 @@
         gazebo="$(arg gazebo)"
         />
+    <!-- D435 camera -->
+    <xacro:property name="camera_pose_file"
+                    value="$(find agimus_demos)/franka/manipulation/config/calibrated-params.yaml" />
+    <xacro:property name="camera_pose" value="${load_yaml(camera_pose_file)}"/>
+    <link name="ref_camera_link"/>
+    <joint name="ref_camera_joint" type="fixed">
+      <parent link="${arm_id}_hand"/>
+      <child link="ref_camera_link"/>
+      <origin xyz="${camera_pose['camera']['x']}
+                   ${camera_pose['camera']['y']}
+                   ${camera_pose['camera']['z']}"
+	      rpy="${camera_pose['camera']['roll']}
+                   ${camera_pose['camera']['pitch']}
+                   ${camera_pose['camera']['yaw']}"/>
+    </joint>
+    <xacro:include filename="$(find realsense2_description)/urdf/_d435.urdf.xacro" />
+    <xacro:sensor_d435 parent="ref_camera_link" name="camera" use_nominal_extrinsics="true">
+      <origin xyz="0 0 0" rpy="0 0 0"/>
+    </xacro:sensor_d435>
+    <xacro:if value="$(arg gazebo)">
+      <xacro:include filename="$(find agimus_demos)/urdf/_d435.gazebo.xacro"/>
+      <xacro:gazebo_d435 camera_name="d435" reference_link="ref_camera_link"
+                         topics_ns="camera"
+                         depth_optical_frame="camera_depth_optical_frame"
+                         color_optical_frame="camera_color_optical_frame"
+                         infrared1_optical_frame="camera_infrared1_optical_frame"
+                         infrared2_optical_frame="camera_infrared2_optical_frame">
+      </xacro:gazebo_d435>
+    </xacro:if>
     <!-- Define additional Gazebo tags -->
     <xacro:if value="$(arg gazebo)">

Commit message: [urdf] Add camera support and rename ref_camera_[link|joint]
  into panda1_ref_camera_[link|joint].

File: urdf/franka_robot.xacro (robot description, xacro)
@@ -26,8 +26,8 @@
                     value="$(find agimus_demos)/franka/manipulation/config/calibrated-params.yaml" />
     <xacro:property name="camera_pose" value="${load_yaml(camera_pose_file)}"/>
-    <link name="ref_camera_link"/>
-    <joint name="ref_camera_joint" type="fixed">
+    <link name="${arm_id}_ref_camera_link"/>
+    <joint name="${arm_id}_ref_camera_joint" type="fixed">
       <parent link="${arm_id}_hand"/>
-      <child link="ref_camera_link"/>
+      <child link="${arm_id}_ref_camera_link"/>
       <origin xyz="${camera_pose['camera']['x']}
                    ${camera_pose['camera']['y']}
@@ -38,10 +38,36 @@
     </joint>
     <xacro:include filename="$(find realsense2_description)/urdf/_d435.urdf.xacro" />
-    <xacro:sensor_d435 parent="ref_camera_link" name="camera" use_nominal_extrinsics="true">
+    <xacro:sensor_d435 parent="${arm_id}_ref_camera_link" name="camera" use_nominal_extrinsics="true">
       <origin xyz="0 0 0" rpy="0 0 0"/>
     </xacro:sensor_d435>
+    <!-- camera support -->
+    <link name="${arm_id}_camera_support_link">
+      <inertial>
+        <mass value="0.010"/>
+        <origin xyz="0 0 0"/>
+        <inertia ixx="0.001" iyy="0.001" izz="0.001" ixy="0" iyz="0" ixz="0"/>
+      </inertial>
+      <visual>
+        <origin xyz="0.022 -0.102 0.036" rpy="3.141592653589793 0 -1.5707963267948966"/>
+        <geometry>
+          <mesh filename="package://agimus_demos/franka/manipulation/meshes/camera-support.stl" scale="0.001 0.001 0.001"/>
+        </geometry>
+      </visual>
+      <collision>
+        <origin xyz="0.022 -0.102 0.036" rpy="3.141592653589793 0 -1.5707963267948966"/>
+        <geometry>
+          <mesh filename="package://agimus_demos/franka/manipulation/meshes/camera-support.stl" scale="0.001 0.001 0.001"/>
+        </geometry>
+      </collision>
+    </link>
+    <joint name="${arm_id}_camera_support_joint" type="fixed">
+      <parent link="${arm_id}_hand"/>
+      <child link="${arm_id}_camera_support_link"/>
+      <origin xyz="0 0 0" rpy="0 0 0"/>
+    </joint>
     <xacro:if value="$(arg gazebo)">
       <xacro:include filename="$(find agimus_demos)/urdf/_d435.gazebo.xacro"/>
-      <xacro:gazebo_d435 camera_name="d435" reference_link="ref_camera_link"
+      <xacro:gazebo_d435 camera_name="d435"
+                         reference_link="${arm_id}_ref_camera_link"
                          topics_ns="camera"
                          depth_optical_frame="camera_depth_optical_frame"

Commit message: [calibration] Collect data for hand eye calibration and compute camera pose.

File: urdf/franka_robot.xacro (robot description, xacro)
@@ -49,5 +49,5 @@
       </inertial>
       <visual>
-        <origin xyz="0.022 -0.102 0.036" rpy="3.141592653589793 0 -1.5707963267948966"/>
+        <origin xyz="0.022 -0.102 -0.035" rpy="3.141592653589793 0 -1.5707963267948966"/>
         <geometry>
           <mesh filename="package://agimus_demos/franka/manipulation/meshes/camera-support.stl" scale="0.001 0.001 0.001"/>
@@ -55,5 +55,5 @@
       </visual>
       <collision>
-        <origin xyz="0.022 -0.102 0.036" rpy="3.141592653589793 0 -1.5707963267948966"/>
+        <origin xyz="0.022 -0.102 -0.035" rpy="3.141592653589793 0 -1.5707963267948966"/>
         <geometry>
           <mesh filename="package://agimus_demos/franka/manipulation/meshes/camera-support.stl" scale="0.001 0.001 0.001"/>
@@ -64,5 +64,5 @@
       <parent link="${arm_id}_hand"/>
       <child link="${arm_id}_camera_support_link"/>
-      <origin xyz="0 0 0" rpy="0 0 0"/>
+      <origin xyz="0 0 0" rpy="3.141592653589793 0 0"/>
     </joint>
     <xacro:if value="$(arg gazebo)">
